Commit message: Change change change

File: rosbot_description/models/rosbot_base/components/orbbec_astra.gazebo.xacro (robot description, xacro)
@@ -33,5 +33,5 @@
     </joint>
     <joint name="orbbec_astra_depth_link_refference_joint" type="fixed">
-      <origin xyz="0.0 0.0 0.0" rpy="${pi/2} ${-pi/2} 0.0" />
+      <origin xyz="0.0 0.0 0.0" rpy="0.0 ${-pi/2} 0.0" />
       <parent link="orbbec_astra_depth_link" />
       <child link="orbbec_astra_depth_refference_link" />
